Commit message: values fixed, no more absolute mesh values

File: robot/arm/models/bimanual_humanoid.urdf (robot description, URDF)
Before this commit: robot bimanual_piper_description, 23 links, 22 joints
Links:
- link cony_text: geometry visual mesh filename=cony_text.STL scale=0.001 0.001 0.001
- link left_base_link: geometry collision mesh filename=base_link.STL; visual mesh filename=base_link.STL
- link left_gripper_base: geometry collision mesh filename=gripper_base.STL; visual mesh filename=gripper_base.STL
- link left_link1: geometry collision mesh filename=link1.STL; visual mesh filename=link1.STL
- link left_link2: geometry collision mesh filename=link2.STL; visual mesh filename=link2.STL
- link left_link3: geometry collision mesh filename=link3.STL; visual mesh filename=link3.STL
- link left_link4: geometry collision mesh filename=link4.STL; visual mesh filename=link4.STL
- link left_link5: geometry collision mesh filename=link5.STL; visual mesh filename=link5.STL
- link left_link6: geometry collision mesh filename=link6.STL; visual mesh filename=link6.STL
- link left_link7: geometry collision mesh filename=link7.STL; visual mesh filename=link7.STL
- link left_link8: geometry collision mesh filename=link8.STL; visual mesh filename=link8.STL
- link right_base_link: geometry collision mesh filename=base_link.STL; visual mesh filename=base_link.STL
- link right_gripper_base: geometry collision mesh filename=gripper_base.STL; visual mesh filename=gripper_base.STL
- link right_link1: geometry collision mesh filename=link1.STL; visual mesh filename=link1.STL
- link right_link2: geometry collision mesh filename=link2.STL; visual mesh filename=link2.STL
- link right_link3: geometry collision mesh filename=link3.STL; visual mesh filename=link3.STL
- link right_link4: geometry collision mesh filename=link4.STL; visual mesh filename=link4.STL
- link right_link5: geometry collision mesh filename=link5.STL; visual mesh filename=link5.STL
- link right_link6: geometry collision mesh filename=link6.STL; visual mesh filename=link6.STL
- link right_link7: geometry collision mesh filename=link7.STL; visual mesh filename=link7.STL
- link right_link8: geometry collision mesh filename=link8.STL; visual mesh filename=link8.STL
- link torso_link: geometry collision mesh filename=torso.STL scale=0.001 0.001 0.001; visual mesh filename=torso.STL scale=0.001 0.001 0.001

Commit message: cony first urdf ready

File: robot/arm/models/bimanual_humanoid.urdf (robot description, URDF)
Before this commit: robot bimanual_piper_description, 23 links, 22 joints
Links:
- added link lift_base, mass 1.0; collision box size=0.118 0.118 0.3; visual box size=0.118 0.118 0.3
- added link lift_bottom_plate; collision box size=0.294 0.294 0.004; visual box size=0.294 0.294 0.004
- added link lift_middle, mass 0.8; collision box size=0.108 0.108 0.208; visual box size=0.108 0.108 0.208
- added link lift_top, mass 0.6; collision box size=0.1 0.1 0.208; visual box size=0.1 0.1 0.208
- added link lift_top_plate; collision box size=0.294 0.294 0.004; visual box size=0.294 0.294 0.004
- link torso_link: geometry collision mesh filename=torso.STL scale=0.001 0.001 0.001; visual box size=0.10033 0.2921 0.10414
Joints:
- added joint lift_base_joint: type fixed, parent lift_bottom_plate, child lift_base, origin xyz=0 0 0.152 rpy=0 0 0
- added joint lift_bottom_plate_joint: type fixed, parent base_link, child lift_bottom_plate, origin xyz=0 0 0 rpy=0 0 0
- added joint lift_middle_joint: type prismatic, parent lift_base, child lift_middle, origin xyz=0 0 0.046 rpy=0 0 0, axis 0 0 1, limit lower=0 upper=0.208 effort=1000 velocity=0.5
- added joint lift_top_joint: type prismatic, parent lift_middle, child lift_top, origin xyz=0 0 0.0 rpy=0 0 0, axis 0 0 1, limit lower=0 upper=0.208 effort=1000 velocity=0.5
- added joint lift_top_plate_joint: type fixed, parent lift_top, child lift_top_plate, origin xyz=0 0 0.106 rpy=0 0 0
- joint torso_joint: origin xyz=0 0 0 rpy=0 0 0 -> xyz=0 0 0.05407 rpy=0 0 0; parent base_link -> lift_top_plate

Commit message: cony head added

File: robot/arm/models/bimanual_humanoid.urdf (robot description, URDF)
Before this commit: robot cony, 28 links, 27 joints
Links:
- added link cony_head; visual mesh filename=cony_head.STL scale=0.001 0.001 0.001
Joints:
- added joint cony_head_joint: type fixed, parent torso_link, child cony_head, origin xyz=0 0 0.05207 rpy=0 0 0

Commit message: fix gripper joints, remove reduced_robot

File: robot/arm/models/bimanual_humanoid.urdf (robot description, URDF)
Before this commit: robot cony, 29 links, 28 joints
Joints:
- joint left_joint7: axis 0 0 1 -> (none); limit lower=0 upper=0.035 effort=10 velocity=1 -> (none); type prismatic -> fixed
- joint left_joint8: axis 0 0 -1 -> (none); limit lower=-0.035 upper=0 effort=10 velocity=1 -> (none); type prismatic -> fixed
- joint right_joint7: axis 0 0 1 -> (none); limit lower=0 upper=0.035 effort=10 velocity=1 -> (none); type prismatic -> fixed
- joint right_joint8: axis 0 0 -1 -> (none); limit lower=-0.035 upper=0 effort=10 velocity=1 -> (none); type prismatic -> fixed

File: robot/arm/models/piper-right.urdf (robot description, URDF)
Before this commit: robot piper_description, 10 links, 9 joints
Links:
- link base_link: geometry collision mesh filename=base_link.STL; visual mesh filename=base_link.STL
- link gripper_base: geometry collision mesh filename=gripper_base.STL; visual mesh filename=gripper_base.STL
- link link1: geometry collision mesh filename=link1.STL; visual mesh filename=link1.STL
- link link2: geometry collision mesh filename=link2.STL; visual mesh filename=link2.STL
- link link3: geometry collision mesh filename=link3.STL; visual mesh filename=link3.STL
- link link4: geometry collision mesh filename=link4.STL; visual mesh filename=link4.STL
- link link5: geometry collision mesh filename=link5.STL; visual mesh filename=link5.STL
- link link6: geometry collision mesh filename=link6.STL; visual mesh filename=link6.STL
- link link7: geometry collision mesh filename=link7.STL; visual mesh filename=link7.STL
- link link8: geometry collision mesh filename=link8.STL; visual mesh filename=link8.STL

Commit message: switched to single prismatic joint for lift at this commit!

File: robot/arm/models/bimanual_humanoid.urdf (robot description, URDF)
Before this commit: robot cony, 29 links, 28 joints
Links:
- removed link lift_middle
- link lift_top: geometry collision box size=0.1 0.1 0.3; visual box size=0.1 0.1 0.3
Joints:
- removed joint lift_middle_joint
- removed joint lift_top_joint
- added joint lift_joint: type prismatic, parent lift_base, child lift_top, origin xyz=0 0 0.0 rpy=0 0 0, axis 0 0 1, limit lower=0 upper=0.3 effort=1000 velocity=0.5
- joint lift_top_plate_joint: origin xyz=0 0 0.106 rpy=0 0 0 -> xyz=0 0 0.152 rpy=0 0 0

Commit message: move ee_left and fix arm velocities

File: robot/arm/models/bimanual_humanoid.urdf (robot description, URDF)
Before this commit: robot cony, 28 links, 27 joints
Links:
- added link ee_left
Joints:
- added joint left_ee_joint: type fixed, parent left_link6, child ee_left, origin xyz=0 0 0.13 rpy=0 -1.5708 0
- joint left_joint1: limit lower=-2.618 upper=0.25 effort=100 velocity=5 -> lower=-2.618 upper=0.25 effort=100 velocity=3.14
- joint left_joint2: limit lower=0 upper=3.14 effort=100 velocity=5 -> lower=0 upper=3.14 effort=100 velocity=3.4
- joint left_joint3: limit lower=-2.967 upper=0 effort=100 velocity=5 -> lower=-2.967 upper=0 effort=100 velocity=3.14
- joint left_joint4: limit lower=-1.745 upper=1.745 effort=100 velocity=5 -> lower=-1.745 upper=1.745 effort=100 velocity=3.9
- joint left_joint5: limit lower=-1.22 upper=1.22 effort=100 velocity=5 -> lower=-1.22 upper=1.22 effort=100 velocity=3.9
- joint left_joint6: limit lower=-2.0944 upper=2.0944 effort=100 velocity=3 -> lower=-2.0944 upper=2.0944 effort=100 velocity=3.9
- joint lift_joint: limit lower=0 upper=0.3 effort=1000 velocity=0.5 -> lower=0 upper=0.3 effort=100 velocity=0.05
- joint right_joint1: limit lower=-0.25 upper=2.618 effort=100 velocity=5 -> lower=-0.25 upper=2.618 effort=100 velocity=3.14
- joint right_joint2: limit lower=0 upper=3.14 effort=100 velocity=5 -> lower=0 upper=3.14 effort=100 velocity=3.4
- joint right_joint3: limit lower=-2.967 upper=0 effort=100 velocity=5 -> lower=-2.967 upper=0 effort=100 velocity=3.14
- joint right_joint4: limit lower=-1.745 upper=1.745 effort=100 velocity=5 -> lower=-1.745 upper=1.745 effort=100 velocity=3.9
- joint right_joint5: limit lower=-1.22 upper=1.22 effort=100 velocity=5 -> lower=-1.22 upper=1.22 effort=100 velocity=3.9
- joint right_joint6: limit lower=-2.0944 upper=2.0944 effort=100 velocity=3 -> lower=-2.0944 upper=2.0944 effort=100 velocity=3.9

Commit message: rename to coney

File: robot/arm/models/bimanual_humanoid.urdf (robot description, URDF)
Before this commit: robot cony, 29 links, 28 joints
Links:
- removed link cony_head
- removed link cony_text
- added link coney_head; visual mesh filename=coney_head.STL scale=0.001 0.001 0.001
Joints:
- removed joint cony_head_joint
- removed joint cony_text_joint
- added joint coney_head_joint: type fixed, parent torso_link, child coney_head, origin xyz=0 0 0.05207 rpy=0 0 0
