Commit message: got all the pieces together - need to make them work

File: robot/arm/models/piper-left.urdf (robot description, URDF)
Before this commit: robot piper_description, 10 links, 9 joints
Joints:
- joint joint1: limit lower=-2.618 upper=2.168 effort=100 velocity=5 -> lower=-2.618 upper=0.0 effort=100 velocity=5

Commit message: graceful shutdown impl

File: robot/arm/models/piper-left.urdf (robot description, URDF)
Before this commit: robot piper_description, 10 links, 9 joints
Joints:
- joint joint1: limit lower=-2.618 upper=0.0 effort=100 velocity=5 -> lower=-2.618 upper=0.25 effort=100 velocity=5

File: robot/arm/models/piper-right.urdf (robot description, URDF)
Before this commit: robot piper_description, 10 links, 9 joints
Joints:
- joint joint1: limit lower=0.0 upper=2.618 effort=100 velocity=5 -> lower=-0.25 upper=2.618 effort=100 velocity=5

Commit message: arm controllers working again

File: robot/arm/models/piper-left.urdf (robot description, URDF)
Before this commit: robot piper_description, 10 links, 9 joints
Joints:
- joint joint6: limit lower=-2.0944 upper=2.0944 effort=100 velocity=3 -> lower=-2.7944 upper=1.4 effort=100 velocity=3; origin xyz=8.8259E-05 -0.091 0 rpy=1.5708 0 0 -> xyz=8.8259E-05 -0.091 0 rpy=1.5708 -0.7 0
